File: schematic/E-bike.kicad_sch (KiCad schematic)
At the start: 18 parts, among them U1 DS3231

Commit message: stuff
Parts:
- added C3, C4: 100n, symbol Device:C
Connections:
- net GND: now also C3.2
- net at 5V. (VOUT), A1.27 (+5V), C2.1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: now also C4.1
- net at Twist_Throttle. (GND), VESC6_MKVI. (VCC): now also Thumb_Throttle. (GND)
- net at 5V. (VOUT), C2.2: now also C4.2
- new net: 5V. (VOUT), C1.1, C3.1, VESC6_MKVI. (VCC)
- new net: Twist_Throttle. (GND), VESC6_MKVI. (VCC)
- new net: Thumb_Throttle. (GND), Twist_Throttle. (GND), VESC6_MKVI. (VCC)
- new net: BLDC_Hall. (V+), VESC6_MKVI. (VCC) (x8)
- new net: VESC6_MKVI. (VCC), VESC_NRF. (VCC) (x6)
Other:
- moved on the sheet: 5V
